Commit message: feeding,laptop,lightswitch,reach updated reset

File: assistive_gym/envs/assets/door/slider_door.urdf (robot description, URDF)
Before this commit: robot on_switch.urdf, 2 links, 1 joints
Links:
- removed link case_link
- removed link on_button_link
- added link door_link, mass 100; collision mesh filename=slider_door.obj; visual mesh filename=slider_door.obj
- added link frame_link, mass 100; collision mesh filename=slider_frame.obj; visual mesh filename=slider_frame.obj
Joints:
- removed joint fixed
- added joint hinge: type prismatic, parent frame_link, child child_link, axis 1 0 0, limit lower=0 upper=.1 effort=100 velocity=100

File: assistive_gym/envs/assets/light_switch/off_switch.urdf (robot description, URDF)
Before this commit: robot on_switch.urdf, 2 links, 1 joints
Links:
- link case_link: mass None -> 5
- link off_button_link: mass None -> 5
