Commit message: combined version 1 and originals, updated Laptop, started LightSwitch

File: assistive_gym/envs/assets/laptop/laptop.urdf (robot description, URDF)
Before this commit: robot laptop.urdf, 2 links, 1 joints
Links:
- link base_link: mass .05 -> 5; geometry collision mesh filename=body_visual.dae; visual mesh filename=body_visual.dae
- link screen_link: mass .01 -> 1; geometry collision mesh filename=screen_visual.dae; visual mesh filename=screen_visual.dae

File: assistive_gym/envs/assets/table/table_tall.urdf (robot description, URDF)
Before this commit: robot table.urdf, 1 links, 0 joints
Links:
- link baseLink: geometry collision mesh filename=table.obj scale=1.5 1 0.05; visual mesh filename=table.obj scale=0.08 0.08 0.7

Commit message: levers

File: assistive_gym/envs/assets/laptop/laptop.urdf (robot description, URDF)
Before this commit: robot laptop.urdf, 2 links, 1 joints
Links:
- link base_link: mass 5 -> None
- link screen_link: mass 1 -> None
Joints:
- joint hinge: limit lower=0 upper=3.14 effort=100 velocity=100 -> lower=-.2 upper=3.14 effort=100 velocity=100; origin (none) -> xyz=1.1 0 .5 rpy=0 0 0

Commit message: lever environments

File: assistive_gym/envs/assets/laptop/laptop.urdf (robot description, URDF)
Before this commit: robot laptop.urdf, 2 links, 1 joints
Joints:
- joint hinge: limit lower=-.2 upper=3.14 effort=100 velocity=100 -> lower=-.2 upper=1.7 effort=100 velocity=100

File: assistive_gym/envs/assets/light_switch/switch.urdf (robot description, URDF)
Before this commit: robot switch.urdf, 2 links, 1 joints
Links:
- link button_link: geometry collision mesh filename=switch.obj scale=5 5 3; visual mesh filename=switch.obj scale=5 5 3
- link case_link: geometry collision mesh filename=case1.obj scale=1 1 .75; visual mesh filename=case1.obj scale=1 1 .75
Joints:
- joint hinge: axis 0 1 0 -> 1 0 0; limit lower=0 upper=3.14 effort=100 velocity=100 -> lower=-1 upper=.1 effort=100 velocity=100; origin xyz=0 0 0 rpy=0 0 0 -> xyz=0 -.3 0 rpy=0 0 0
